Commit message: del testing.cpp

File: src/ur5_with_gripper/urdf/ur5_with_gripper.urdf (robot description, URDF)
Before this commit: robot ur5_with_gripper, 13 links, 12 joints
Joints:
- joint tcp_joint: origin xyz=0 0 0.12 rpy=0 0 0 -> xyz=0 0 0.07 rpy=0 0 0

Commit message: changed to only calculate trajectory one time

File: src/ur5_with_gripper/urdf/ur5_with_gripper.urdf (robot description, URDF)
Before this commit: robot ur5_with_gripper, 13 links, 12 joints
Joints:
- joint tcp_joint: origin xyz=0 0 0.07 rpy=0 0 0 -> xyz=0 0 0.15 rpy=0 0 0

Commit message: tool has been changed

File: src/ur5_with_gripper/urdf/ur5_with_gripper.urdf (robot description, URDF)
Before this commit: robot ur5_with_gripper, 13 links, 12 joints
Joints:
- joint gripper_joint: origin xyz=0 0 0 rpy=0 0 1.57079632679 -> xyz=0 0 0.04 rpy=1.570796326794897 0 1.570796326794897
- joint tcp_joint: origin xyz=0 0 0.15 rpy=0 0 0 -> xyz=0 0.15 0 rpy=0 0 0

Commit message: Fixed launch file

File: src/ur5_with_gripper/urdf/ur5_with_gripper.urdf (robot description, URDF)
Before this commit: robot ur5_with_gripper, 13 links, 12 joints
Joints:
- joint gripper_joint: origin xyz=0 0 0.04 rpy=1.570796326794897 0 1.570796326794897 -> xyz=0 0 0 rpy=1.5708 0 0.0
- joint shoulder_pan_joint: limit lower=-3.14159265359 upper=3.14159265359 effort=150.0 velocity=3.15 -> lower=-6.14159265359 upper=6.14159265359 effort=150.0 velocity=3.15
- joint tcp_joint: origin xyz=0 0.15 0 rpy=0 0 0 -> xyz=0 0 0.15 rpy=0 0 0

Commit message: Fixed URDF

File: src/ur5_with_gripper/urdf/ur5_with_gripper.urdf (robot description, URDF)
Before this commit: robot ur5_with_gripper, 13 links, 12 joints
Joints:
- joint elbow_joint: limit lower=-3.14159265359 upper=3.14159265359 effort=150.0 velocity=3.15 -> lower=-6.14159265359 upper=6.14159265359 effort=150.0 velocity=3.15
- joint gripper_joint: origin xyz=0 0 0 rpy=1.5708 0 0.0 -> xyz=0 0 0.04 rpy=1.570796326794897 0 1.570796326794897
- joint shoulder_lift_joint: limit lower=-3.14159265359 upper=3.14159265359 effort=150.0 velocity=3.15 -> lower=-6.14159265359 upper=6.14159265359 effort=150.0 velocity=3.15
- joint tcp_joint: origin xyz=0 0 0.15 rpy=0 0 0 -> xyz=0 0.15 0 rpy=0 0 0
- joint wrist_1_joint: limit lower=-3.14159265359 upper=3.14159265359 effort=28.0 velocity=3.2 -> lower=-6.14159265359 upper=6.14159265359 effort=28.0 velocity=3.2
- joint wrist_2_joint: limit lower=-3.14159265359 upper=3.14159265359 effort=28.0 velocity=3.2 -> lower=-6.14159265359 upper=6.14159265359 effort=28.0 velocity=3.2
- joint wrist_3_joint: limit lower=-3.14159265359 upper=3.14159265359 effort=28.0 velocity=3.2 -> lower=-6.14159265359 upper=6.14159265359 effort=28.0 velocity=3.2

Commit message: changed throwing angle to 45 deg

File: src/ur5_with_gripper/urdf/ur5_with_gripper.urdf (robot description, URDF)
Before this commit: robot ur5_with_gripper, 13 links, 12 joints
Joints:
- joint tcp_joint: origin xyz=0 0.15 0 rpy=0 0 0 -> xyz=0 0.18 0 rpy=0 0 0
